File: TFT_LCD_Display_EC11_Board.kicad_pcb (KiCad board)
At the start: 2 copper layers, 91 x 44 mm, 29 parts, among them J2 Control, J3 I2C, J4 TFT-LCD-DISPLAY-EC11, J5 USB_C_Receptacle_USB2.0_16P, Q1 BC848, Q2 BC848, U1 LM2937-3.3V, U2 USBLC6-2SC6, U3 ESP32-WROVER-E-N4R8, U4 CP2104

Commit message: Tweede Commit
Parts:
- renumbered J5 to J1, R7 to R1, R8 to R2, TP4 to TP3, TP5 to TP4, TP6 to TP5
Connections:
- J1 pad SH: (no net) -> GND
Other:
- board text added: "(5V)"
- board text added: "ADW2604"
- board text added: "By Willem Aandewiel"
- board text added: "Ext.Trgr"
- board text added: "OUTPUT"
- board text added: "Piggy Back Board TFT LCD Display EC11"
- board text added: "RESET"
- board text added: "Rev.1.0 [21-04-2026]"

Commit message: Add 3D/openSCAD
Routing:
- net 3v3: track 163.5 -> 166.4 mm
Changed lines of the file:
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@@
 	)
 	(segment
-		(start 169.3 121)
-		(end 183.76 121)
+		(start 187 113.4)
+		(end 188.66 115.06)
 		(width 0.2)
 		(layer "F.Cu")
@@
 	)
 	(segment
-		(start 183.76 121)
+		(start 188.66 115.06)
 		(end 189.7 115.06)
+		(width 0.2)
+		(layer "F.Cu")
+		(net "3v3")
+	)
+	(segment
+		(start 169.3 121)
+		(end 169.3 118.4)
 		(width 0.2)
 		(layer "F.Cu")
@@
 	)
 	(segment
+		(start 169.3 118.4)
+		(end 174.3 113.4)
+		(width 0.2)
+		(layer "F.Cu")
+		(net "3v3")
+	)
+	(segment
 		(start 122.3549 110.6549)
 		(end 121.3 109.6)
@@
 		(width 0.2)
 		(layer "F.Cu")
+		(net "3v3")
+	)
+	(segment
+		(start 174.3 113.4)
+		(end 187 113.4)
+		(width 0.2)
+		(layer "F.Cu")

Commit message: Combine Rev 2.0 and openSCAD files
Parts:
- removed TP4: RTS, TestPoint:TestPoint_Loop_D3.80mm_Drill2.0mm
- removed TP5: DTR, TestPoint:TestPoint_Loop_D3.80mm_Drill2.0mm
- added C4: 100nF, Capacitor_SMD:C_1206_3216Metric_Pad1.33x1.80mm_HandSolder, F.Cu at (157.5, 91.9)
- added C5: 100nF, Capacitor_SMD:C_1206_3216Metric_Pad1.33x1.80mm_HandSolder, F.Cu at (123.1, 98.0)
- added C6: 100nF, Capacitor_SMD:C_1206_3216Metric_Pad1.33x1.80mm_HandSolder, F.Cu at (123.1, 113.5)
- added D1: 3v3, LED_SMD:LED_1206_3216Metric_Pad1.42x1.75mm_HandSolder, F.Cu at (181.8, 85.5)
- added JP2: U2-, Jumper:SolderJumper-2_P1.3mm_Open_RoundedPad1.0x1.5mm, F.Cu at (114.3, 108.5)
- added JP3: 5Volt, Jumper:SolderJumper-2_P1.3mm_Open_RoundedPad1.0x1.5mm, F.Cu at (145.0, 111.8)
- added R10: 10k, Resistor_SMD:R_1206_3216Metric_Pad1.30x1.75mm_HandSolder, F.Cu at (141.6, 107.5)
- added R7: 10k, Resistor_SMD:R_1206_3216Metric_Pad1.30x1.75mm_HandSolder, F.Cu at (115.0, 93.5)
- added R8: 10k, Resistor_SMD:R_1206_3216Metric_Pad1.30x1.75mm_HandSolder, F.Cu at (115.0, 85.0)
- added R9: 10k, Resistor_SMD:R_1206_3216Metric_Pad1.30x1.75mm_HandSolder, F.Cu at (134.9, 107.5)
- added SW1: BOOT, Button_Switch_SMD:SW_SPST_FSMSM, F.Cu at (146.5, 91.6)
- added SW2: EN, Button_Switch_SMD:SW_SPST_FSMSM, F.Cu at (153.5, 91.6)
- C3: footprint Capacitor_SMD:C_0805_2012Metric_Pad1.18x1.45mm_HandSolder -> Capacitor_SMD:C_1206_3216Metric_Pad1.33x1.80mm_HandSolder
- J1: moved to B.Cu
- JP1: value 5Volt -> U2+
- R1: value 5k1 -> 2k; footprint Resistor_SMD:R_0805_2012Metric_Pad1.20x1.40mm_HandSolder -> Resistor_SMD:R_1206_3216Metric_Pad1.30x1.75mm_HandSolder
- R2: value 5k1 -> 220R; footprint Resistor_SMD:R_0805_2012Metric_Pad1.20x1.40mm_HandSolder -> Resistor_SMD:R_1206_3216Metric_Pad1.30x1.75mm_HandSolder
- R3: value 10k -> 220R
- R4, R5: value 10k -> 5k1
- TP1, TP2, TP3: footprint TestPoint:TestPoint_Loop_D3.80mm_Drill2.0mm -> TestPoint:TestPoint_Loop_D2.50mm_Drill1.0mm
- U1: value LM2937-3.3V -> MCP1826S; footprint Package_TO_SOT_SMD:SOT-223 -> Package_TO_SOT_SMD:SOT-223-3_TabPin2
- U3: footprint myNewLibrary:XCVR_ESP32-WROVER-E-N4R8 -> MyNewLibrary:ESP32-WROVER-B-E
- U4: value CP2104 -> CH340C; footprint Package_DFN_QFN:QFN-24-1EP_4x4mm_P0.5mm_EP2.6x2.6mm -> Package_SO:SOIC-16_3.9x9.9mm_P1.27mm
- moved R1 77.9 mm to (184.5, 85.5), turned to -90 degrees
- moved R2 41.0 mm to (146.4, 100.0), turned to 180 degrees
- moved TP2 34.0 mm to (106.0, 91.0)
- moved R3 31.7 mm to (153.4, 100.0)
- moved JP1 31.1 mm to (114.2, 101.5), turned to 0 degrees
- moved C3 25.6 mm to (133.6, 86.5), turned to 0 degrees
- moved R4 23.2 mm to (107.0, 111.5)
- moved U1 17.2 mm to (123.2, 89.5), turned to 180 degrees
- moved C2 16.8 mm to (135.2, 91.0), turned to 0 degrees
- moved R5 15.6 mm to (107.5, 95.5), turned to 0 degrees
- moved TP1 10.0 mm to (106.0, 116.5)
- moved U3 7.25 mm to (169.5, 98.3), turned to 0 degrees
- moved J1 5.93 mm to (107.9, 106.5), turned to 90 degrees
- moved U4 4.81 mm to (122.9, 105.6)
- moved TP3 4.68 mm to (111.0, 116.5)
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Connections:
- JP1 pad 1: Net-(J2-Pin_1) -> D+
- JP1 pad 2: VBUS -> Net-(JP1-B)
- Q1 pad 2: DTR -> ~{DTR}
- Q2 pad 2: RTS -> ~{RTS}
- R1 pad 1: Net-(J1-CC1) -> Net-(D1-A)
- R1 pad 2: GND -> 3v3
- R2 pad 1: Net-(J1-CC2) -> Net-(R2-Pad1)
- R2 pad 2: GND -> GPIO0
- R3 pad 1: 3v3 -> Net-(R3-Pad1)
- R3 pad 2: Net-(U4-~{RST}) -> ~{ENABLE}
- R4 pad 1: RTS -> Net-(J1-CC1)
- R4 pad 2: Net-(Q1-B) -> GND
- R5 pad 1: DTR -> Net-(J1-CC2)
- R5 pad 2: Net-(Q2-B) -> GND
- R6 pad 1: EXT-TRIGGER -> GPIO0
- U2 pad 1: D- -> D+
- U2 pad 3: D+ -> D-
- U2 pad 4: Net-(U4-D+) -> Net-(JP2-B)
- U2 pad 6: Net-(U4-D-) -> Net-(JP1-B)
- U4 pad 1: unconnected-(U4-~{RI}-Pad1) -> GND
- U4 pad 13: unconnected-(U4-RXT/GPIO.1-Pad13) -> ~{DTR}
- U4 pad 14: unconnected-(U4-TXT/GPIO.0-Pad14) -> ~{RTS}
- U4 pad 16: unconnected-(U4-VPP-Pad16) -> VBUS
- U4 pad 2: GND -> ESP-RX
- U4 pad 3: Net-(U4-D+) -> ESP-TX
- U4 pad 4: Net-(U4-D-) -> Net-(U4-V3)
- U4 pad 5: 3v3 -> Net-(JP1-B)
- U4 pad 6: 3v3 -> Net-(JP2-B)
- U4 pad 7: 3v3 -> unconnected-(U4-NC-Pad7)
- U4 pad 8: VBUS -> unconnected-(U4-NC-Pad8)
- U4 pad 9: Net-(U4-~{RST}) -> unconnected-(U4-~{CTS}-Pad9)
Routing:
- net DC: track 56.5 -> 20.8 mm, vias 1 -> 0
- net RTS: track 34.2 -> 0.00 mm, vias 3 -> 0
- net 3v3: track 166.4 -> 199.5 mm
- net ~{DTR}: track 0.00 -> 31.0 mm, vias 0 -> 2
- net CS: track 42.8 -> 12.6 mm, vias 1 -> 0
- net DTR: track 25.5 -> 0.00 mm
- net VBUS: track 77.7 -> 100.9 mm, vias 3 -> 1
- net ~{RTS}: track 0.00 -> 22.4 mm, vias 0 -> 2
- net ESP-TX: track 44.2 -> 63.8 mm, vias 0 -> 2
- net SDA: track 69.2 -> 51.4 mm
- net ESP-RX: track 47.3 -> 62.7 mm, vias 0 -> 2
- net OUTPUT: track 47.5 -> 33.5 mm, vias 1 -> 0
- net BLK: track 18.6 -> 32.5 mm, vias 0 -> 1
- net GPIO0: track 79.7 -> 91.5 mm, vias 0 -> 2
- net SCL: track 70.7 -> 60.2 mm
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Other:
- board text added: "A"
- board text added: "K"
- board text added: "Rev.2.0 [06-05-2026]"
- board text removed: "Rev.1.0 [21-04-2026]"
